Commit message: merge gazebo sim capability into movement controller

File: description.xacro (robot description, xacro)
@@ -1,7 +1,7 @@
-<?xml version="1.0" encoding="UTF-8"?>
+<?xml version="1.0"?>
 <robot xmlns:xacro="http://wiki.ros.org/xacro" name="$(arg name)">
   <!-- robot name parameter -->
   <xacro:arg name="name" default="ur"/>
-  <xacro:include filename="$(find movement_controller)/srdf/ur_macro.srdf.xacro"/>
-  <xacro:ur_srdf/>
+  <!-- create link fixed to the "world" -->
+  <link name="world" />
 </robot>

File: src/movement_controller/srdf/ur/ur.srdf.xacro (robot description, xacro)
@@ -1,8 +1,10 @@
 <?xml version="1.0" encoding="UTF-8"?>
-<robot xmlns:xacro="http://wiki.ros.org/xacro">
+<robot xmlns:xacro="http://wiki.ros.org/xacro" name="$(arg name)">
 <!--This does not replace URDF, and is not an extension of URDF.
     This is a format for representing semantic information about the robot structure.
     A URDF file must exist for this robot as well, where the joints and the links that are referenced are defined
 -->
+  <!-- robot name parameter -->
+  <xacro:arg name="name" default="ur"/>
   <xacro:macro name="ur_srdf" params="">
     <!--GROUPS - Representation of a set of joints and links. This can be useful for specifying DOF to plan for, defining arms, end effectors, etc-->
@@ -37,4 +39,7 @@
     <disable_collisions link1="wrist_1_link" link2="wrist_3_link" reason="Never" />
     <disable_collisions link1="wrist_2_link" link2="wrist_3_link" reason="Adjacent" />
+    <disable_collisions link1="ground_plane" link2="base_link" reason="Adjacent" />
+    <disable_collisions link1="ground_plane" link2="base_link_inertia" reason="Adjacent" />
   </xacro:macro>
+  <xacro:ur_srdf/>
 </robot>
