Commit message: create station package; move urdf, srdf, world and models

File: src/station/config/urdf/ur/gz_sim.urdf.xacro (robot description, xacro)
@@ -71,11 +71,11 @@
       <origin xyz="0 0 0" rpy="0 0 0"/>
       <geometry>
-        <mesh filename="file:///workspaces/movement_controller/model/station/meshes/station_visual.dae"/>
-      </geometry>
-    </visual>
-    <collision>
-      <origin xyz="0 0 0" rpy="0 0 0"/>
-      <geometry>
-        <mesh filename="file:///workspaces/movement_controller/model/station/meshes/station_collision.stl"/>
+        <mesh filename="file://$(find station)/config/model/station/meshes/station_visual.dae"/>
+      </geometry>
+    </visual>
+    <collision>
+      <origin xyz="0 0 0" rpy="0 0 0"/>
+      <geometry>
+        <mesh filename="file://$(find station)/config/model/station/meshes/station_collision.stl"/>
       </geometry>
     </collision>
@@ -112,11 +112,11 @@
       <origin xyz="0 0 0" rpy="0 0 0"/>
       <geometry>
-        <mesh filename="file:///workspaces/movement_controller/model/tool_mount/meshes/tool_mount_with_camera_visual.dae"/>
-      </geometry>
-    </visual>
-    <collision>
-      <origin xyz="0 0 0" rpy="0 0 0"/>
-      <geometry>
-        <mesh filename="file:///workspaces/movement_controller/model/tool_mount/meshes/tool_mount_with_camera_collision.stl"/>
+        <mesh filename="file://$(find station)/config/model/tool_mount/meshes/tool_mount_with_camera_visual.dae"/>
+      </geometry>
+    </visual>
+    <collision>
+      <origin xyz="0 0 0" rpy="0 0 0"/>
+      <geometry>
+        <mesh filename="file://$(find station)/config/model/tool_mount/meshes/tool_mount_with_camera_collision.stl"/>
       </geometry>
     </collision>
@@ -183,11 +183,11 @@
       <origin xyz="0 0 0" rpy="0 0 0"/>
       <geometry>
-        <mesh filename="file:///workspaces/movement_controller/model/conveyor/meshes/conveyor_visual.dae"/>
-      </geometry>
-    </visual>
-    <collision>
-      <origin xyz="0 0 0" rpy="0 0 0"/>
-      <geometry>
-        <mesh filename="file:///workspaces/movement_controller/model/conveyor/meshes/conveyor_collision.stl"/>
+        <mesh filename="file://$(find station)/config/model/conveyor/meshes/conveyor_visual.dae"/>
+      </geometry>
+    </visual>
+    <collision>
+      <origin xyz="0 0 0" rpy="0 0 0"/>
+      <geometry>
+        <mesh filename="file://$(find station)/config/model/conveyor/meshes/conveyor_collision.stl"/>
       </geometry>
     </collision>

File: src/station/config/urdf/ur/real.urdf.xacro (robot description, xacro)
@@ -84,5 +84,5 @@
       <origin xyz="0 0 0" rpy="0 0 0"/>
       <geometry>
-        <mesh filename="file:///workspaces/movement_controller/model/station/meshes/station_visual.dae"/>
+        <mesh filename="file://$(find station)/config/model/station/meshes/station_visual.dae"/>
       </geometry>
     </visual>
@@ -90,5 +90,5 @@
       <origin xyz="0 0 0" rpy="0 0 0"/>
       <geometry>
-        <mesh filename="file:///workspaces/movement_controller/model/station/meshes/station_collision.stl"/>
+        <mesh filename="file://$(find station)/config/model/station/meshes/station_collision.stl"/>
       </geometry>
     </collision>
@@ -125,5 +125,5 @@
       <origin xyz="0 0 0" rpy="0 0 0"/>
       <geometry>
-        <mesh filename="file:///workspaces/movement_controller/model/tool_mount/meshes/tool_mount_with_camera_visual.dae"/>
+        <mesh filename="file://$(find station)/config/model/tool_mount/meshes/tool_mount_with_camera_visual.dae"/>
       </geometry>
     </visual>
@@ -131,5 +131,5 @@
       <origin xyz="0 0 0" rpy="0 0 0"/>
       <geometry>
-        <mesh filename="file:///workspaces/movement_controller/model/tool_mount/meshes/tool_mount_with_camera_collision.stl"/>
+        <mesh filename="file://$(find station)/config/model/tool_mount/meshes/tool_mount_with_camera_collision.stl"/>
       </geometry>
     </collision>
@@ -148,5 +148,5 @@
       <origin xyz="0 0 0" rpy="0 0 0"/>
       <geometry>
-        <mesh filename="file:///workspaces/movement_controller/model/conveyor/meshes/conveyor_visual.dae"/>
+        <mesh filename="file://$(find station)/config/model/conveyor/meshes/conveyor_visual.dae"/>
       </geometry>
     </visual>
@@ -154,5 +154,5 @@
       <origin xyz="0 0 0" rpy="0 0 0"/>
       <geometry>
-        <mesh filename="file:///workspaces/movement_controller/model/conveyor/meshes/conveyor_collision.stl"/>
+        <mesh filename="file://$(find station)/config/model/conveyor/meshes/conveyor_collision.stl"/>
       </geometry>
     </collision>
