Commit message: add cameras package

File: src/station/config/srdf/default_setup.srdf.xacro (robot description, xacro)
@@ -7,4 +7,6 @@
   <!-- robot name parameter -->
   <xacro:arg name="name" default="ur"/>
+  <!-- Camera SRDF macro (disables camera<->parent collisions) -->
+  <xacro:include filename="$(find cameras)/srdf/basler.srdf.xacro"/>
   <xacro:macro name="ur_srdf" params="">
     <!--GROUPS - Representation of a set of joints and links. This can be useful for specifying DOF to plan for, defining arms, end effectors, etc-->
@@ -46,4 +48,6 @@
     <disable_collisions link1="tool_mount_link" link2="wrist_2_link" reason="Never" />
     <disable_collisions link1="tool_mount_link" link2="wrist_3_link" reason="Never" />
+    <!-- Disable collisions between the camera and the link it is mounted on -->
+    <xacro:basler_camera_srdf parent="tool_mount_link" name="basler" />
   </xacro:macro>
   <xacro:ur_srdf/>

File: src/station/config/urdf/ur/gz_sim.urdf.xacro (robot description, xacro)
@@ -7,4 +7,5 @@
   <!-- import ros2_control joint control description -->
   <xacro:include filename="$(find ur_description)/urdf/inc/ur_joint_control.xacro" />
+  <xacro:include filename="$(find cameras)/urdf/basler.urdf.xacro"/>
   <!-- ros2_control macro (merged from ur_gz.ros2_control.xacro) -->
   <xacro:macro name="ur_ros2_control" params="
@@ -112,5 +113,5 @@
       <origin xyz="0 0 0" rpy="0 0 0"/>
       <geometry>
-        <mesh filename="file://$(find station)/config/model/tool_mount/meshes/tool_mount_with_camera_visual.dae"/>
+        <mesh filename="file://$(find station)/config/model/tool_mount/meshes/tool_mount_visual.dae"/>
       </geometry>
     </visual>
@@ -118,5 +119,5 @@
       <origin xyz="0 0 0" rpy="0 0 0"/>
       <geometry>
-        <mesh filename="file://$(find station)/config/model/tool_mount/meshes/tool_mount_with_camera_collision.stl"/>
+        <mesh filename="file://$(find station)/config/model/tool_mount/meshes/tool_mount_collision.stl"/>
       </geometry>
     </collision>
@@ -129,53 +130,9 @@
     <parent link="$(arg tf_prefix)tool0"/>
     <child link="tool_mount_link"/>
-    <origin xyz="0 0 0" rpy="0 0 0"/>
+    <origin xyz="0 0 0" rpy="-1.57 -1.57 0"/>
   </joint>
-  <!-- Gazebo (Harmonic / gz-sim) Camera Sensor.
-       Rendering is handled by the gz-sim-sensors-system plugin loaded in the
-       world (default.world). The sensor publishes on a Gazebo Transport topic;
-       it is bridged to ROS 2 via ros_gz_bridge in the launch file.
-       Image topic:       /basler_camera/image
-       CameraInfo topic:  /basler_camera/camera_info (auto, sibling of image) -->
-<gazebo reference="tool_mount_link">
-  <sensor name="basler_camera" type="camera">
-    <pose>0.0700233 -0.127701 -0.0225334 0 0 -1.57</pose>
-    <always_on>true</always_on>
-    <update_rate>30.0</update_rate>
-    <visualize>true</visualize>
-    <topic>/basler_camera/image</topic>
-    <gz_frame_id>tool_mount_link</gz_frame_id>
-    <camera name="basler_camera_sensor">
-      <horizontal_fov>1.0472</horizontal_fov> <!-- ~60 degrees -->
-      <image>
-        <width>1920</width>
-        <height>1080</height>
-        <format>R8G8B8</format>
-      </image>
-      <clip>
-        <near>0.01</near>
-        <far>100.0</far>
-      </clip>
-      <noise>
-        <type>gaussian</type>
-        <mean>0.0</mean>
-        <stddev>0.007</stddev>
-      </noise>
-      <!-- Lens distortion (Brown-Conrady / plumb-bob model, same as OpenCV).
-           k1/k2/k3: radial coefficients  (negative k1 = barrel distortion).
-           p1/p2:    tangential coefficients.
-           center:   normalised distortion centre (0.5 0.5 = optical centre).
-           Tune these to match the real Basler lens calibration output. -->
-      <distortion>
-        <k1>-0.2477771909786335</k1>
-        <k2>0.126037678472415</k2>
-        <k3>-0.0010056044464992401</k3>
-        <p1>0.000391226451080845</p1>
-        <p2>-0.04092116227683235</p2>
-        <center>0.5 0.5</center>
-      </distortion>
-      <optical_frame_id>tool_mount_link</optical_frame_id>
-    </camera>
-  </sensor>
-</gazebo>
+  <xacro:basler_camera parent="tool_mount_link" name="basler" simulated="true" tf_prefix="$(arg tf_prefix)">
+    <origin xyz="-0.03 0.025 -0.057" rpy="1.57 0 1.57"/>
+  </xacro:basler_camera>
   <!-- conveyor belt fixed to world frame -->
   <link name="conveyor">

File: src/station/config/urdf/ur/real.urdf.xacro (robot description, xacro)
@@ -8,4 +8,5 @@
   <xacro:include filename="$(find ur_robot_driver)/urdf/ur.ros2_control.xacro" />
   <xacro:include filename="$(find ur_description)/urdf/inc/ur_transmissions.xacro" />
+  <xacro:include filename="$(find cameras)/urdf/basler.urdf.xacro"/>
   <!-- possible 'ur_type' values: ur3, ur5, ur10, ur3e, ur5e, ur7e, ur10e, ur12e, ur16e, ur8long, ur15, ur18, ur20, ur30 -->
   <!-- the default value should raise an error in case this was called without defining the type -->
@@ -125,5 +126,5 @@
       <origin xyz="0 0 0" rpy="0 0 0"/>
       <geometry>
-        <mesh filename="file://$(find station)/config/model/tool_mount/meshes/tool_mount_with_camera_visual.dae"/>
+        <mesh filename="file://$(find station)/config/model/tool_mount/meshes/tool_mount_visual.dae"/>
       </geometry>
     </visual>
@@ -131,5 +132,5 @@
       <origin xyz="0 0 0" rpy="0 0 0"/>
       <geometry>
-        <mesh filename="file://$(find station)/config/model/tool_mount/meshes/tool_mount_with_camera_collision.stl"/>
+        <mesh filename="file://$(find station)/config/model/tool_mount/meshes/tool_mount_collision.stl"/>
       </geometry>
     </collision>
@@ -142,6 +143,9 @@
     <parent link="$(arg tf_prefix)tool0"/>
     <child link="tool_mount_link"/>
-    <origin xyz="0 0 0" rpy="0 0 0"/>
-  </joint>
+    <origin xyz="0 0 0" rpy="-1.57 -1.57 0"/>
+  </joint>
+  <xacro:basler_camera parent="tool_mount_link" name="basler" simulated="false" tf_prefix="$(arg tf_prefix)">
+    <origin xyz="-0.03 0.025 -0.057" rpy="1.57 0 1.57"/>
+  </xacro:basler_camera>
   <link name="conveyor">
     <visual>

Commit message: add laser cross-sensor and endtool packages

File: src/station/config/srdf/default_setup.srdf.xacro (robot description, xacro)
@@ -9,4 +9,6 @@
   <!-- Camera SRDF macro (disables camera<->parent collisions) -->
   <xacro:include filename="$(find cameras)/srdf/basler.srdf.xacro"/>
+  <xacro:include filename="$(find laser_sensors)/srdf/cross_laser.srdf.xacro"/>
+  <xacro:include filename="$(find endtools)/srdf/dispensing_tool.srdf.xacro"/>
   <xacro:macro name="ur_srdf" params="">
     <!--GROUPS - Representation of a set of joints and links. This can be useful for specifying DOF to plan for, defining arms, end effectors, etc-->
@@ -50,4 +52,13 @@
     <!-- Disable collisions between the camera and the link it is mounted on -->
     <xacro:basler_camera_srdf parent="tool_mount_link" name="basler" />
+    <xacro:basler_camera_srdf parent="flange" name="basler" />
+    <xacro:basler_camera_srdf parent="wrist_3_link" name="basler" />
+    <!-- Disable collisions between the laser sensor and the link it is mounted on -->
+    <xacro:cross_laser_srdf parent="station" name="captron"/>
+    <!-- Disable collisions between the dispensing tool and the link it is mounted on -->
+    <xacro:dispensing_tool_srdf parent="tool_mount_link" name="dispensing"/>
+    <xacro:dispensing_tool_srdf parent="flange" name="dispensing" />
+    <xacro:dispensing_tool_srdf parent="wrist_3_link" name="dispensing" />
+    <xacro:dispensing_tool_srdf parent="basler_camera_link" name="dispensing" />
   </xacro:macro>
   <xacro:ur_srdf/>

File: src/station/config/urdf/ur/gz_sim.urdf.xacro (robot description, xacro)
@@ -8,4 +8,6 @@
   <xacro:include filename="$(find ur_description)/urdf/inc/ur_joint_control.xacro" />
   <xacro:include filename="$(find cameras)/urdf/basler.urdf.xacro"/>
+  <xacro:include filename="$(find laser_sensors)/urdf/cross_laser.urdf.xacro"/>
+  <xacro:include filename="$(find endtools)/urdf/dispensing_tool.urdf.xacro"/>
   <!-- ros2_control macro (merged from ur_gz.ros2_control.xacro) -->
   <xacro:macro name="ur_ros2_control" params="
@@ -92,4 +94,7 @@
     <child link="station"/>
   </joint>
+  <xacro:cross_laser parent="station" name="captron" simulated="true" tf_prefix="$(arg tf_prefix)">
+    <origin xyz="0.35 0.45 0.95" rpy="0 0 3.14"/>
+  </xacro:cross_laser>
   <!-- arm mounted on top of the station (z=1.0) -->
   <xacro:ur_robot
@@ -135,4 +140,7 @@
     <origin xyz="-0.03 0.025 -0.057" rpy="1.57 0 1.57"/>
   </xacro:basler_camera>
+  <xacro:dispensing parent="tool_mount_link" name="dispensing" simulated="true" tf_prefix="$(arg tf_prefix)">
+    <origin xyz="0.0475 0 0" rpy="0 0 0"/>
+  </xacro:dispensing>
   <!-- conveyor belt fixed to world frame -->
   <link name="conveyor">
