Commit message: implement cross laser sensor simulation

File: src/laser_sensors/urdf/cross_laser.urdf.xacro (robot description, xacro)
@@ -8,4 +8,6 @@
     simulated:=true
     update_rate:=30.0
+    window_size:=0.04
+    standoff:=0.0
     *origin">
     <link name="${name}_laser_sensor_link">
@@ -33,4 +35,87 @@
         <xacro:insert_block name="origin"/>
     </joint>
+    <link name="${name}_orl2_intersection"/>
+    <joint name="${name}_orl2_intersection_joint" type="fixed">
+      <parent link="${name}_laser_sensor_link"/>
+      <child link="${name}_orl2_intersection"/>
+      <origin xyz="0 -0.0425 0.02591" rpy="0 0 0"/>
+    </joint>
+    <!--
+      Simulated laser cross.
+      The physical ORL2-40T projects two perpendicular laser lines that meet at
+      a single intersection (the TCP measuring point) inside a ~40 mm window.
+      Each line is modelled here as a single-ray gpu_lidar that fires across the
+      window; an object entering the window returns a short range on both beams.
+      Both beams are centred on the intersection point, which sits at the sensor
+      link origin, optionally pushed out along +Z by 'standoff' metres:
+        * beam_1 fires along the local +X axis
+        * beam_2 fires along the local +Y axis (X-ray rotated 90 deg about Z)
+      Each ray reaches at most 'window_size' metres so a "no object" reading
+      returns +inf (never interrupted) while an object in the window returns a
+      range <= window_size. The node's 'detection_distance' parameter (default
+      0.04 m) decides the interruption threshold.
+    -->
+    <xacro:if value="${simulated}">
+      <gazebo reference="${name}_laser_sensor_link">
+        <sensor name="${name}_beam_1_sensor" type="gpu_lidar">
+          <pose>${-window_size/2.0} -0.0425 ${0.02591+standoff} 0 0 0</pose>
+          <always_on>true</always_on>
+          <update_rate>${update_rate}</update_rate>
+          <visualize>true</visualize>
+          <topic>simulated_laser_cross/beam_x_axis</topic>
+          <gz_frame_id>${name}_laser_sensor_link</gz_frame_id>
+          <lidar>
+            <scan>
+              <horizontal>
+                <samples>1</samples>
+                <resolution>1</resolution>
+                <min_angle>0</min_angle>
+                <max_angle>0</max_angle>
+              </horizontal>
+              <vertical>
+                <samples>1</samples>
+                <resolution>1</resolution>
+                <min_angle>0</min_angle>
+                <max_angle>0</max_angle>
+              </vertical>
+            </scan>
+            <range>
+              <min>0.001</min>
+              <max>${window_size}</max>
+              <resolution>0.0002</resolution>
+            </range>
+          </lidar>
+        </sensor>
+        <sensor name="${name}_beam_2_sensor" type="gpu_lidar">
+          <pose>0 ${-0.0425+(-window_size/2.0)} ${0.02591+standoff} 0 0 ${pi/2.0}</pose>
+          <always_on>true</always_on>
+          <update_rate>${update_rate}</update_rate>
+          <visualize>true</visualize>
+          <topic>simulated_laser_cross/beam_y_axis</topic>
+          <gz_frame_id>${name}_laser_sensor_link</gz_frame_id>
+          <lidar>
+            <scan>
+              <horizontal>
+                <samples>1</samples>
+                <resolution>1</resolution>
+                <min_angle>0</min_angle>
+                <max_angle>0</max_angle>
+              </horizontal>
+              <vertical>
+                <samples>1</samples>
+                <resolution>1</resolution>
+                <min_angle>0</min_angle>
+                <max_angle>0</max_angle>
+              </vertical>
+            </scan>
+            <range>
+              <min>0.001</min>
+              <max>${window_size}</max>
+              <resolution>0.0002</resolution>
+            </range>
+          </lidar>
+        </sensor>
+      </gazebo>
+    </xacro:if>
   </xacro:macro>
 </robot>
